File: pcb/tdb-distributor/tdb-distributor.kicad_sch (KiCad schematic)
At the start: 15 parts, among them J1 Conn_02x07_Odd_Even, J2 Conn_02x07_Odd_Even, J3 Conn_02x07_Odd_Even, J4 Conn_02x07_Odd_Even, J5 Screw_Terminal_01x03, J6 Conn_01x06_Pin, J7 Conn_01x07_Pin, J8 Conn_01x08_Pin, U1 LM317_TO-220

Commit message: Board redesign
Includes R7 MPU and WizNet
Adds buffer chips to hopefully support both sides of the display
Parts:
- removed J6: Conn_01x06_Pin, Connector_PinHeader_2.54mm:PinHeader_1x06_P2.54mm_Vertical, symbol Connector:Conn_01x06_Pin
- removed J7: Conn_01x07_Pin, Connector_PinHeader_2.54mm:PinHeader_1x07_P2.54mm_Vertical, symbol Connector:Conn_01x07_Pin
- removed J8: Conn_01x08_Pin, Connector_PinHeader_2.54mm:PinHeader_1x08_P2.54mm_Vertical, symbol Connector:Conn_01x08_Pin
- added C10, C8: 10n, Capacitor_SMD:C_0603_1608Metric, symbol Device:C
- added C11: 22n, Capacitor_SMD:C_0603_1608Metric, symbol Device:C
- added C12, C13, C3, C4, C5, C9: 4.7u, Capacitor_SMD:C_0603_1608Metric, symbol Device:C
- added C14, C15, C16: 22u, Capacitor_SMD:C_0603_1608Metric, symbol Device:C
- added C6, C7: 18p, Capacitor_SMD:C_0603_1608Metric, symbol Device:C
- added IC1, IC2: 74HC541D,653, Package_SO:SOIC-20W_7.5x12.8mm_P1.27mm, symbol 74HC541D,653:74HC541D,653
- added J6: RJ45_Hanrun_HR911105A_Horizontal, Connector_RJ:RJ45_Hanrun_HR911105A_Horizontal, symbol Connector:RJ45_Hanrun_HR911105A_Horizontal
- added J7: USB_C_Receptacle_USB2.0_16P, Connector_USB:USB_C_Receptacle_G-Switch_GT-USB-7010ASV, symbol Connector:USB_C_Receptacle_USB2.0_16P
- added J8: Conn_01x02, Connector_PinHeader_2.54mm:PinHeader_1x02_P2.54mm_Vertical, symbol Connector_Generic:Conn_01x02
- added R10: 12.4k, Resistor_SMD:R_0603_1608Metric, symbol Device:R
- added R11, R12, R13, R14: 49.9, Resistor_SMD:R_0603_1608Metric, symbol Device:R
- added R15: 10, Resistor_SMD:R_0603_1608Metric, symbol Device:R
- added R16, R17: 100, Resistor_SMD:R_0603_1608Metric, symbol Device:R
- added R18, R2, R20, R21, R3, R4, R5, R6, R7, R8: 5.1k, Resistor_SMD:R_0603_1608Metric, symbol Device:R
- added R19: 100k, Resistor_SMD:R_0603_1608Metric, symbol Device:R
- added R9: 1M, Resistor_SMD:R_0603_1608Metric, symbol Device:R
- added SW_Reset1: SW_Push, Button_Switch_THT:SW_TH_Tactile_Omron_B3F-10xx, symbol Switch:SW_Push
- added U2: W5500, Package_QFP:LQFP-48_7x7mm_P0.5mm, symbol Interface_Ethernet:W5500
- added U3: R7FA4M1AB3CFM, PLQP0064KB-C_REN, symbol R7FA4M1AB3CFM:R7FA4M1AB3CFM
- added Y1: 25M, Crystal:Crystal_SMD_5032-2Pin_5.0x3.2mm, symbol Device:Crystal
- C1: footprint Capacitor_THT:C_Disc_D5.0mm_W2.5mm_P2.50mm -> Capacitor_SMD:C_0603_1608Metric
- C2: footprint Capacitor_THT:CP_Radial_D8.0mm_P2.50mm -> Capacitor_SMD:C_0603_1608Metric
- R1: footprint Resistor_THT:R_Axial_DIN0411_L9.9mm_D3.6mm_P12.70mm_Horizontal -> Resistor_SMD:R_0603_1608Metric
Connections:
- net +5V: now also C12.1, C13.1, C14.1, C15.1, C16.1, IC1.20 (VCC), IC2.20 (VCC), J7.A4 (VBUS), J7.A9 (VBUS), J7.B4 (VBUS), J7.B9 (VBUS), J8.1 (Pin_1), R19.1, R2.1, R4.1, R7.2, R8.2, U3.11 (VCC), U3.21 (VCC_USB_LDO), U3.39 (VCC), U3.55 (P012/VREFH), U3.56 (AVCC0)
- net BCD_A: now also IC1.6 (A4), IC2.6 (A4), U3.41 (P107); no longer J1.5 (Pin_5), J2.5 (Pin_5), J3.5 (Pin_5), J4.5 (Pin_5)
- net BCD_B: now also IC1.7 (A5), IC2.5 (A3), U3.42 (P106); no longer J1.7 (Pin_7), J2.7 (Pin_7), J3.7 (Pin_7), J4.7 (Pin_7)
- net BCD_C: now also IC1.8 (A6), IC2.4 (A2), U3.43 (P105); no longer J1.9 (Pin_9), J2.9 (Pin_9), J3.9 (Pin_9), J4.9 (Pin_9)
- net CLOCK: now also IC1.3 (A1), IC2.9 (A7), U3.36 (P111); no longer J1.1 (Pin_1), J2.1 (Pin_1), J3.1 (Pin_1), J4.1 (Pin_1)
- net DATA_A: now also IC1.4 (A2), IC2.8 (A6), U3.37 (P112); no longer J1.12 (Pin_12), J1.3 (Pin_3), J2.12 (Pin_12), J2.3 (Pin_3)
- net DATA_B: now also IC1.5 (A3), IC2.7 (A5), U3.38 (P113); no longer J3.12 (Pin_12), J3.3 (Pin_3), J4.12 (Pin_12), J4.3 (Pin_3)
- net GND: now also C10.1, C11.2, C12.2, C13.2, C14.2, C15.2, C16.2, C3.2, C4.2, C5.2, C6.2, C7.2, C8.2, C9.2, IC1.1 (~{OE1}), IC1.10 (GND), IC1.19 (~{OE2}), IC1.2 (A0), IC2.1 (~{OE1}), IC2.10 (GND), IC2.19 (~{OE2}), IC2.2 (A0), J6.8, J6.SH, J7.A1 (GND), J7.A12 (GND), J7.B1 (GND), J7.B12 (GND), J7.S1 (SHIELD), R10.2, R18.2, R20.2, R21.2, R3.2, R6.2, SW_Reset1.1, U2.14 (AGND), U2.16 (AGND), U2.19 (AGND), U2.23 (RSVD), U2.29 (GND), U2.3 (AGND), U2.48 (AGND), U2.9 (AGND), U3.17 (VSS_USB), U3.40 (VSS), U3.57 (AVSS0), U3.8 (VSS); no longer J1.11 (Pin_11), J2.11 (Pin_11), J3.11 (Pin_11), J4.11 (Pin_11)
- net STROBE: now also IC1.9 (A7), IC2.3 (A1), U3.44 (P104); no longer J1.13 (Pin_13), J2.13 (Pin_13), J3.13 (Pin_13), J4.13 (Pin_13)
- new net: R8.1, U3.27 (P200)
- new net: J7.B5 (CC2), R18.1
- new net: J6.12, R16.1
- new net: C9.1, U2.20 (TOCAP)
- new net: C11.1, J6.4 (TCT), R15.2
- new net: R4.2, R5.1, U3.16 (P407)
- new net: C10.2, J6.5 (RCT), R12.2, R14.2
- new net: C6.1, R9.1, U2.30 (XI/CLKIN), Y1.1
- new net: C7.1, R9.2, U2.31 (XO), Y1.2
- new net: R5.2, R6.1
- new net: R19.2, R20.1, U3.49 (P500)
- new net: J6.9, R17.1
- new net: R7.1, U3.26 (P201/MD)
- new net: C4.1, U3.5 (VCL)
- new net: J8.2 (Pin_2), R21.1, U3.63 (P001)
- new net: J7.A5 (CC1), R3.1
- new net: R10.1, U2.10 (EXRES1)
- new net: C8.1, U2.22 (1V2O)
- new net +3.3V: C3.1, C5.1, R11.1, R13.1, R15.1, R16.2, R17.2, U2.11 (AVDD), U2.15 (AVDD), U2.17 (AVDD), U2.21 (AVDD), U2.28 (VDD), U2.36 (~{INT}), U2.4 (AVDD), U2.43 (PMODE2), U2.44 (PMODE1), U2.45 (PMODE0), U2.8 (AVDD), U3.20 (VCC_USB), U3.4 (VBATT)
- new net ACTLED: J6.10, U2.27 (ACTLED)
- new net ETH_CS: U2.32 (~{SCS}), U3.45 (P103)
- new net ETH_RESET: U2.37 (~{RST}), U3.47 (P101)
- new net LINKLED: J6.11, U2.25 (LINKLED)
- new net RESET: R2.2, SW_Reset1.2, U3.25 (RES)
- new net RXIN: J6.6 (RD-), R14.1, U2.6 (RXP)
- new net RXIP: J6.3 (RD+), R12.1, U2.5 (RXN)
- new net SPI_CLK: U2.33 (SCLK), U3.46 (P102)
- new net SPI_MISO: U2.34 (MISO), U3.13 (P410)
- new net SPI_MOSI: U2.35 (MOSI), U3.12 (P411)
- new net TXON: J6.2 (TD-), R13.2, U2.2 (TXP)
- new net TXOP: J6.1 (TD+), R11.2, U2.1 (TXN)
- new net USBD+: J7.A6 (D+), J7.B6 (D+), U3.19 (P914/USB_DP)
- new net USBD-: J7.A7 (D-), J7.B7 (D-), U3.18 (P915/USB_DM)
- new net aBCD_A: IC1.14 (Y4), J3.5 (Pin_5), J4.5 (Pin_5)
- new net aBCD_B: IC1.13 (Y5), J3.7 (Pin_7), J4.7 (Pin_7)
- new net aBCD_C: IC1.12 (Y6), J3.9 (Pin_9), J4.9 (Pin_9)
- new net aCLOCK: IC1.17 (Y1), J3.1 (Pin_1), J4.1 (Pin_1)
- new net aDATA_A: IC1.16 (Y2), J3.12 (Pin_12), J3.3 (Pin_3)
- new net aDATA_B: IC1.15 (Y3), J4.12 (Pin_12), J4.3 (Pin_3)
- new net aSTROBE: IC1.11 (Y7), J3.13 (Pin_13), J4.13 (Pin_13)
- new net bBCD_A: IC2.14 (Y4), J1.5 (Pin_5), J2.5 (Pin_5)
- new net bBCD_B: IC2.15 (Y3), J1.7 (Pin_7), J2.7 (Pin_7)
- new net bBCD_C: IC2.16 (Y2), J1.9 (Pin_9), J2.9 (Pin_9)
- new net bCLOCK: IC2.11 (Y7), J1.1 (Pin_1), J2.1 (Pin_1)
- new net bDATA_A: IC2.12 (Y6), J1.12 (Pin_12), J1.3 (Pin_3)
- new net bDATA_B: IC2.13 (Y5), J2.12 (Pin_12), J2.3 (Pin_3)
- new net bSTROBE: IC2.17 (Y1), J1.13 (Pin_13), J2.13 (Pin_13)
Other:
- moved on the sheet: C1, C2, J5, R1, RV1, TP1, U1
